File: acoustic-carrier-hw/acoustic-carrier-board/fpga-config-flash.kicad_sch (KiCad schematic)
At the start: 20 parts, among them IC1 ECP5-BGA256, J701 Conn_02x06_Odd_Even, J703 Conn_02x06_Odd_Even, U701 W25Q128JVS, U702 W25Q128JVS

Commit message: Did big ig parts of routing (next) make sure to re-add pull-ups/downs accordingly
Parts:
- removed J701, J703: Conn_02x06_Odd_Even, Connector_PinSocket_2.54mm:PinSocket_2x06_P2.54mm_Horizontal, symbol Connector_Generic:Conn_02x06_Odd_Even
- added J701: Conn_02x07_Odd_Even, Connector_PinSocket_2.54mm:PinSocket_2x07_P2.54mm_Vertical, symbol Connector_Generic:Conn_02x07_Odd_Even
- added J702: Conn_02x09_Odd_Even, Connector_PinSocket_2.54mm:PinSocket_2x09_P2.54mm_Vertical, symbol Connector_Generic:Conn_02x09_Odd_Even
Connections:
- net FPGA_CFG0: now also J701.2 (Pin_2)
- net FPGA_CFG1: now also RN701.3 (R3.1), J701.4 (Pin_4); no longer RN702.1 (R1.1)
- net FPGA_CFG2: now also RN701.2 (R2.1), J701.6 (Pin_6); no longer R703.2
- net FPGA_DONE: now also J701.5 (Pin_5)
- net FPGA_RESET: now also RN702.1 (R1.1), J701.1 (Pin_1); no longer RN702.4 (R4.1)
- net GND: now also J701.11 (Pin_11)
- net JTAG.TCK: now also J701.12 (Pin_12); no longer R701.1
- net JTAG.TDI: now also R701.1, J701.8 (Pin_8); no longer RN701.2 (R2.1)
- net JTAG.TDO: now also J701.14 (Pin_14); no longer RN701.3 (R3.1)
- net JTAG.TMS: now also J701.10 (Pin_10)
- net QSPI.CSPPIn1: now also RN703.3 (R3.1), J702.16 (Pin_16); no longer RN704.3 (R3.1)
- net QSPI.CSPPIn2: now also RN703.4 (R4.1), J702.14 (Pin_14); no longer RN704.1 (R1.1)
- net QSPI.CSn: now also J702.12 (Pin_12); no longer RN704.4 (R4.1)
- net QSPI.D0: now also J702.17 (Pin_17)
- net QSPI.D1: now also RN704.4 (R4.1), J702.15 (Pin_15); no longer RN703.2 (R2.1)
- net QSPI.D2: now also RN704.3 (R3.1), J702.13 (Pin_13); no longer RN703.3 (R3.1)
- net QSPI.D3: now also RN704.1 (R1.1), J702.11 (Pin_11); no longer RN703.4 (R4.1)
- net QSPI.MCLK: now also RN703.2 (R2.1), J702.18 (Pin_18); no longer R704.2
- net VCORE_3V3: now also J701.13 (Pin_13)
- net ~{FPGA_INIT}: now also R703.2, J701.3 (Pin_3); no longer RN702.3 (R3.1)
- net FPGA_ADC_LED0: now reaches IC1.M9 (~{WRITE}/PB18A)
- net FPGA_ADC_LED0: now also RN702.4 (R4.1), J701.9 (Pin_9)
- net FPGA_ADC_LED1: now reaches IC1.P8 (~{CS1}/PB13B)
- net FPGA_ADC_LED1: now also RN702.3 (R3.1), J701.7 (Pin_7)
- new net: J702.9 (Pin_9), R704.2
- no-connect marks 16 -> 17
Other:
- moved on the sheet: C701, C702, C703
