File: acoustic-carrier-hw/acoustic-carrier-board/ethernet-phy.kicad_sch (KiCad schematic)
At the start: 50 parts, among them J1201 HR911130A, U1201 KSZ9031RN, Y1201 25MHz

Commit message: [carrier] Added extra decoupling to ADC bias voltage
Parts:
- removed TP1201: TestPoint, TestPoint:TestPoint_Loop_D1.80mm_Drill1.0mm_Beaded, symbol Connector:TestPoint
Changed lines of the file:
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@@
 	)
 	(junction
-		(at 203.2 247.65)
-		(diameter 0)
-		(color 0 0 0 0)
-	)
-	(junction
 		(at 228.6 92.71)
 		(diameter 0)
@@
 	(wire
 		(pts
-			(xy 203.2 246.38) (xy 203.2 247.65)
-		)
-		(stroke
-			(width 0)
-			(type default)
-		)
-	)
-	(wire
-		(pts
 			(xy 125.73 46.99) (xy 125.73 44.45)
 		)
@@
 	(wire
 		(pts
-			(xy 189.23 247.65) (xy 203.2 247.65)
+			(xy 189.23 247.65) (xy 212.09 247.65)
 		)
 		(stroke
@@
 	(wire
 		(pts
-			(xy 203.2 247.65) (xy 212.09 247.65)
-		)
-		(stroke
-			(width 0)
-			(type default)
-		)
-	)
-	(wire
-		(pts
 			(xy 241.3 45.72) (xy 246.38 45.72)
 		)
@@
 					(unit 1)
 				)
-			)
-		)
-	)
-	(symbol
-		(lib_id "Connector:TestPoint")
-		(at 203.2 246.38 0)
-		(unit 1)
-		(exclude_from_sim no)
-		(in_bom yes)
-		(on_board yes)
-		(dnp no)
-		(property "Reference" "TP1201"
-			(at 203.962 237.998 0)
-			(effects
-				(font
-					(size 1.27 1.27)
-				)
-				(justify left)
-			)
-		)
-		(property "Value" "TestPoint"
-			(at 203.708 240.284 0)
-			(effects
-				(font
-					(size 1.27 1.27)
-				)
-				(justify left)
-			)
-		)
-		(property "Footprint" "TestPoint:TestPoint_Loop_D1.80mm_Drill1.0mm_Beaded"
-			(at 208.28 246.38 0)
-			(effects
-				(font
-					(size 1.27 1.27)
-				)
-				(hide yes)
-			)
-		)
-		(property "Datasheet" "~"
-			(at 208.28 246.38 0)
-			(effects
-				(font
-					(size 1.27 1.27)
-				)
-				(hide yes)
-			)
-		)
-		(property "Description" "test point"
-			(at 203.2 246.38 0)
-			(effects
-				(font
-					(size 1.27 1.27)
-				)
-				(hide yes)
-			)
-		)
-		(pin "1"
-		)
-		(instances
-			(project "acoustic-carrier-board"
-				(path "/25b015c9-ab13-4427-b72c-b6f348597100/d85f0c18-d011-408e-9192-d89f0585c7ff"
-					(reference "TP1201")
-					(unit 1)
-				)
