File: acoustic-carrier-hw/acoustic-carrier-board/fpga-bank-01.kicad_sch (KiCad schematic)
At the start: 12 parts, among them IC1 ECP5-BGA256, Y401 Crystal Oscillator

Commit message: [carrier] finished for production (next) reroute the LPDDR3, with appropriate CMD-CTRL bus delays, and change banks for command-control
Parts:
- IC1: Manufacturer Lattice -> (none)
