File: acoustic-piezodriver-hw/acoustic-piezodriver-board/inverter.kicad_sch (KiCad schematic)
At the start: 52 parts, among them J3 Conn_02x08_Odd_Even, U11 TMP102xxDRL, U12 TMP102xxDRL, U13 AMS1117-3.3, U2 UCC27282DR, U3 UCC27282DR, U6 NCE6005AS, U7 NCE6005AS

Commit message: [piezodriver] Reorganised piezodriver schematic (next) figure out output filtering
Parts:
- removed C13, C14, C18, C19, C5, C7: 1uF, Capacitor_SMD:C_0805_2012Metric, symbol Device:C_Small
- removed C15, C20, C21: 220uF, Capacitor_THT:C_Radial_D10.0mm_H16.0mm_P5.00mm, symbol Device:C_Polarized_Small
- removed C54: 22uF, Capacitor_SMD:C_0805_2012Metric, symbol Device:C_Small
- removed C55, C56: 10nF, Capacitor_SMD:C_0402_1005Metric, symbol Device:C_Small
- removed D12, D13: RED, Diode_SMD:D_0603_1608Metric, symbol Device:LED_Small
- removed D4: SS510, Diode_SMD:D_SMA, symbol Device:D_Schottky_Small
- removed J3: Conn_02x08_Odd_Even, Connector_PinHeader_2.54mm:PinHeader_2x08_P2.54mm_Horizontal, symbol Connector_Generic:Conn_02x08_Odd_Even
- removed R36, R38, R40: 4.7k, Resistor_SMD:R_0402_1005Metric, symbol Device:R_Small
- removed R37, R43: 1k, Resistor_SMD:R_0402_1005Metric, symbol Device:R_Small
- removed U11, U12: TMP102xxDRL, Package_TO_SOT_SMD:SOT-563, symbol Sensor_Temperature:TMP102xxDRL
- removed U13: AMS1117-3.3, Package_TO_SOT_SMD:SOT-223-3_TabPin2, symbol Regulator_Linear:AMS1117-3.3
- removed U2, U3: UCC27282DR, Package_SO:SOIC-8-1EP_3.9x4.9mm_P1.27mm_EP2.29x3mm, symbol ucc27282:UCC27282DR
- added P201: WJ128V-5.0-3P, iw-connector:WJ128V-5.0-3P, symbol iw-connector:WJ128V-5.0-3P
- added U201, U202: UCC27282DR, Package_SO:SOIC-8-1EP_3.9x4.9mm_P1.27mm_EP2.29x3mm, symbol iw-power:UCC27282DR
Connections:
- net +VDC is gone; now on net VDC: R10.2, R7.2, U6.7 (D2), U6.8 (D2), U7.7 (D2), U7.8 (D2)
- net GND: now also P201.3, U201.7 (VSS), U202.7 (VSS)
- net at D9.1 (K), R4.2: now also U202.8 (LO)
- net at D10.1 (K), R2.1: now also U201.8 (LO)
- net at C1.1: now also U202.2 (HB)
- net at D8.1 (K), R3.2: now also U202.3 (HO)
- net at D11.1 (K), R1.2: now also U201.3 (HO)
- net at C2.1: now also U201.2 (HB)
- net +10V renamed VDC
- net VDC: now also U201.1 (VDD), U202.1 (VDD)
- net INV_LOAD0 renamed INV_LOADN
- net INV_LOADN: now also P201.2, U201.4 (HS)
- net INV_LOAD1 renamed INV_LOADP
- net INV_LOADP: now also P201.1, U202.4 (HS)
- new net PWM.0_HI: U201.5 (HI)
- new net PWM.0_LI: U201.6 (LI)
- new net PWM.1_HI: U202.5 (HI)
- new net PWM.1_LI: U202.6 (LI)
Other:
- added sheet INVERTER_POWER (INVERTER_POWER.kicad_sch)
- note removed: "Address, check Table 6-4 - One ADD0 high - One with ADD0 low Pull-ups - SDA, SCL: open-drain LED - Vf: 2 V, I = 1.2 mA (when ok)"
- note removed: "BOOST BYPASS"
- note removed: "DECOUPLING AND BULK"
- note removed: "If boost is inactive -> directly pass input to inverter"
- note removed: "Inverter voltage not necessarily equal to input voltage!"
- note removed: "PWM CONNECTORS"
- note removed: "Peak frequency capacitors 20 A over 15 ns with dV = 0.2 V => 1.5 uF"
- note removed: "Pins: - SDA, SCL (2) + gnd (2) - PWM (4) + GND (4) - BOOST_EN + SEPIC_EN (2) (basically DC so no ground needed here) So: 8 pins with ground connected"
- note removed: "Polymer Bulk capacitors 3 Amps RMS over 600 ns Irms-peak currrent: 2.65 A each"
- note removed: "TEMPERATURE REGULATION"
- note removed: "Vin_max: 15V"
- note removed: "WARN: DIAMETER PHI_D(10) x L(15) - Should be the same as 10x20, different height - Check with manufacturer"
- moved on the sheet: C1, C10, C11, C12, C2, C3, C4, C6, C8, C9, D10, D11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
